File: TTG.kicad_pcb (KiCad board)
At the start: 2 copper layers, 100 x 100 mm, 223 parts, among them J1 RF_In, J10 Conn_01x01, J11 Conn_01x01, J12 Conn_01x01, J13 Conn_01x01, J14 RF_In, J15 IF, J2 Jack-DC, J3 RF_In, J4 RF_In, J5 RF_In, J6 RF_In, J7 RF_In, J8 OFF, J9 OFF, Q1 MMBT9018, Q10 MMBTFJ310, Q2 MMBT9018, Q3 MMBT9018, Q4 MMBT9018, Q5 SS9018, Q6 MMBTFJ310, Q7 MMBTFJ310, Q8 MMBTFJ310, Q9 MMBTFJ310, SW1 SW_DPDT_x2, SW2 SW_DPDT_x2, SW3 SW_DPDT_x2, SW4 SW_DPDT_x2, SW5 SW_DPDT_x2, SW6 SW_DPDT_x2, SW7 SW_DPDT_x2, SW8 SW_DPDT_x2, T1 Transformer, T10 Transformer_1P_2S, T11 Transformer, T13 Transformer, T2 Transformer, T3 Transformer_1P_1S, T4 Transformer_1P_2S, T5 Transformer_1P_2S, T6 Transformer_1P_2S, T7 Transformer_1P_2S, T8 Transformer_1P_2S, T9 Transformer_1P_2S, U1 L7809, U2 NC7WZ14, U3 FSA3157L6X, U4 FSA3157L6X, U5 LM317L_TO92, U6 L78L05_TO92, U7 FSA3157L6X, U8 FSA3157L6X, Y1 Crystal_GND23, Y2 Crystal_GND23

Commit message: SC2314
Parts:
- added C56: 100nF, TTG:C_1206_0603, F.Cu at (108.1, 105.9)
- added C57: 100nF, TTG:C_1206_0603, F.Cu at (133.1, 92.2)
- added C58: 100nF, TTG:C_1206_0603, F.Cu at (130.8, 125.3)
- added C59: 100nF, TTG:C_1206_0603, F.Cu at (124.9, 116.3)
- added C60: 100nF, TTG:C_1206_0603, F.Cu at (123.2, 93.0)
- added C61: 100nF, TTG:C_1206_0603, F.Cu at (139.7, 100.8)
- added C62: 100nF, TTG:C_1206_0603, F.Cu at (134.6, 80.0)
- added C63: 100nF, TTG:C_1206_0603, F.Cu at (146.5, 78.5)
- added C64: 100nF, TTG:C_1206_0603, F.Cu at (135.5, 83.8)
- added C65: 100nF, TTG:C_1206_0603, F.Cu at (118.6, 77.7)
- added C66: 100nF, TTG:C_1206_0603, F.Cu at (124.2, 71.9)
- added C67: 100nF, TTG:C_1206_0603, F.Cu at (115.1, 67.0)
- added C68: 100nF, TTG:C_1206_0603, F.Cu at (112.3, 76.7)
- added D1: 1N4001, Diodes_ThroughHole:D_DO-41_SOD81_P7.62mm_Horizontal, F.Cu at (140.9, 104.3)
- added D10: LL4148, Diodes_SMD:D_MiniMELF_Handsoldering, F.Cu at (128.6, 89.5)
- added D6: LL4148, Diodes_SMD:D_MiniMELF_Handsoldering, F.Cu at (119.7, 37.7)
- added D7: LL4148, Diodes_SMD:D_MiniMELF_Handsoldering, F.Cu at (119.7, 41.0)
- added D8: LL4148, Diodes_SMD:D_MiniMELF_Handsoldering, F.Cu at (98.7, 75.6)
- added D9: LL4148, Diodes_SMD:D_MiniMELF_Handsoldering, F.Cu at (127.5, 69.3)
- added J16: RX/TX, Pin_Headers:Pin_Header_Straight_1x02_Pitch2.54mm, F.Cu at (92.1, 75.6)
- added L10: 100uH, Resistors_ThroughHole:R_Axial_DIN0204_L3.6mm_D1.6mm_P7.62mm_Horizontal, F.Cu at (118.6, 74.4)
- added L8: 100uH, Resistors_ThroughHole:R_Axial_DIN0204_L3.6mm_D1.6mm_P7.62mm_Horizontal, F.Cu at (122.3, 78.3)
- added L9: 100uH, Resistors_ThroughHole:R_Axial_DIN0204_L3.6mm_D1.6mm_P7.62mm_Horizontal, F.Cu at (121.5, 69.4)
- added Q11: SI2301-TP, TO_SOT_Packages_SMD:SOT-23_Handsoldering, F.Cu at (102.4, 70.1)
- added Q12: SI2301-TP, TO_SOT_Packages_SMD:SOT-23_Handsoldering, F.Cu at (94.0, 70.1)
- added Q13: BF998, TO_SOT_Packages_SMD:SOT-143_Handsoldering, F.Cu at (126.7, 120.7)
- added Q14: SC2314, TO_SOT_Packages_THT:TO-126_Horizontal, F.Cu at (134.9, 77.0)
- added R100: 100R, TTG:R_1206_0603, F.Cu at (134.8, 126.5)
- added R101: 2.2k, Resistors_SMD:R_1206_HandSoldering, F.Cu at (124.9, 126.0)
- added R102: 100R, TTG:R_1206_0603, F.Cu at (127.4, 116.2)
- added R103: 5.1k, TTG:R_1206_0603, F.Cu at (124.7, 80.7)
- added R104: 100, TTG:R_1206_0603, F.Cu at (131.8, 73.9)
- added R105: 5.1k, TTG:R_1206_0603, F.Cu at (143.8, 73.4)
- added R106: 100, TTG:R_1206_0603, F.Cu at (139.2, 80.0)
- added R107: 100, TTG:R_1206_0603, F.Cu at (143.8, 78.5)
- added R95: 1k, TTG:R_1206_0603, F.Cu at (119.6, 115.2)
- added R96: 100, TTG:R_1206_0603, F.Cu at (139.4, 93.0)
- added R97: 100, TTG:R_1206_0603, F.Cu at (122.6, 100.8)
- added R98: 470, TTG:R_1206_0603, F.Cu at (128.5, 125.3)
- added R99: 27k, TTG:R_1206_0603, F.Cu at (131.8, 116.2)
- added T12: FEEDBACK, TTG:TF_2, F.Cu at (130.6, 63.9)
- added T14: Transformer_1P_2S, TTG:HF_transf3, F.Cu at (129.2, 109.1)
- added T15: Transformer_1P_2S, TTG:HF_transf3, F.Cu at (127.7, 98.3)
- added T16: FEEDBACK, TTG:TF_2, F.Cu at (129.0, 85.6)
- added T17: Transformer, TTG:TF14, F.Cu at (139.2, 83.3)
- added U9: FSA3157L6X, TO_SOT_Packages_SMD:SOT-363_SC-70-6_Handsoldering, F.Cu at (123.2, 97.0)
- C14: footprint RX998:C_1206_0603 -> Capacitors_SMD:C_1206_HandSoldering
- C30: value 10uF -> 100nF; footprint Capacitors_Tantalum_SMD:CP_Tantalum_Case-A_EIA-3216-18_Hand -> TTG:C_1206_0603
- R75, R76: value 100 -> 1k
- R78: value 10k -> 100
- R79: value 10k -> 1k
- T10: value Transformer_1P_2S -> N7ZWY1_4; footprint TTG:HF_transf3 -> TTG:N7ZWY
- T9: value Transformer_1P_2S -> Transformer_1P_1S; footprint TTG:HF_transf3 -> TTG:TF14
- moved C49 98.3 mm to (109.5, 42.1), turned to 90 degrees
- moved C50 98.1 mm to (112.8, 42.1), turned to 90 degrees
- moved L7 94.5 mm to (109.5, 46.0), turned to 270 degrees
- moved C39 94.3 mm to (89.9, 50.0), turned to 270 degrees
- moved L6 94.2 mm to (112.8, 46.0), turned to 270 degrees
- moved C38 93.0 mm to (94.8, 50.0), turned to 270 degrees
- moved C35 89.3 mm to (89.9, 55.4), turned to 90 degrees
- moved C36 87.8 mm to (94.8, 55.4), turned to 90 degrees
- moved L4 87.4 mm to (92.3, 56.5), turned to 90 degrees
- moved L3 86.1 mm to (97.2, 56.5), turned to 90 degrees
- moved C52 83.0 mm to (109.5, 57.5), turned to 270 degrees
- moved C51 82.7 mm to (112.8, 57.5), turned to 270 degrees
- moved R81 80.3 mm to (104.0, 61.0), turned to 90 degrees
- moved C42 79.9 mm to (106.5, 61.0), turned to 270 degrees
- moved L5 77.4 mm to (101.0, 64.5)
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Connections:
- C30 pad 1: Net-(C30-Pad1) -> GND
- C30 pad 2: GND -> Net-(C30-Pad2)
- C33 pad 1: Net-(C30-Pad1) -> GND
- C33 pad 2: GND -> Net-(C30-Pad2)
- R75 pad 1: Net-(C30-Pad1) -> +6V
- R75 pad 2: Net-(R75-Pad2) -> Net-(C30-Pad2)
- R76 pad 1: Net-(R76-Pad1) -> Net-(C30-Pad2)
- R76 pad 2: LO -> GND
- R78 pad 1: +6V -> Net-(R78-Pad1)
- R78 pad 2: Net-(C30-Pad1) -> Net-(R78-Pad2)
- R79 pad 1: Net-(C30-Pad1) -> +6V
- R79 pad 2: GND -> Net-(R78-Pad1)
- R92 pad 2: (no net) -> Net-(D8-Pad2)
- T10 pad 1: RF -> Net-(C34-Pad2)
- T10 pad 2: GND -> RF
- T10 pad 4: Net-(C34-Pad2) -> Net-(T10-Pad4)
- T10 pad 5: Net-(C34-Pad2) -> Net-(T10-Pad5)
- T10 pad 6: Net-(T10-Pad6) -> Net-(T10-Pad4)
- T9 pad 1: IF -> Net-(T10-Pad3)
- T9 pad 2: GND -> IF
- T9 pad 3: Net-(T9-Pad3) -> Net-(T10-Pad5)
- T9 pad 4: Net-(R75-Pad2) -> IF
- U7 pad 1: Net-(T10-Pad3) -> Net-(T10-Pad5)
- U7 pad 3: Net-(T10-Pad6) -> Net-(T10-Pad3)
- U7 pad 4: Net-(T9-Pad6) -> Net-(C30-Pad2)
- U8 pad 1: Net-(T10-Pad6) -> Net-(T15-Pad6)
- U8 pad 3: Net-(T10-Pad3) -> Net-(T15-Pad3)
- U8 pad 4: Net-(T9-Pad3) -> Net-(T14-Pad3)
- U8 pad 6: Net-(R76-Pad1) -> Net-(R96-Pad1)
Routing:
- net +6V: track 0.00 -> 130.3 mm, vias 0 -> 4
- net IF: track 0.00 -> 124.7 mm, vias 0 -> 1
- net +12V: track 0.00 -> 90.2 mm, vias 0 -> 2
- net RX: track 0.00 -> 63.7 mm, vias 0 -> 3
- net Net-(C6-Pad1): track 0.00 -> 55.4 mm, vias 0 -> 2
- net +5V: track 0.00 -> 51.0 mm, vias 0 -> 2
- net Net-(C2-Pad1): track 0.00 -> 48.1 mm
- net TX: track 0.00 -> 46.7 mm
- net Net-(C1-Pad2): track 0.00 -> 42.0 mm
- net VXO: track 0.00 -> 36.7 mm, vias 0 -> 2
- net Net-(C21-Pad2): track 0.00 -> 36.6 mm
- net GND: track 0.00 -> 35.7 mm, vias 0 -> 17
- net Net-(C31-Pad1): track 0.00 -> 30.4 mm
- net Net-(C47-Pad1): track 0.00 -> 29.9 mm, vias 0 -> 4
- net Net-(Q10-Pad2): track 0.00 -> 26.8 mm
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- added copper zone on B.Cu, net GND
- added copper zone on F.Cu, net GND

Commit message: release, no rasin mixer
Parts:
- removed C30, C63, C64, C65, C66, C67, C68: 100nF, TTG:C_1206_0603
- removed D10, D9: LL4148, Diodes_SMD:D_MiniMELF_Handsoldering
- removed L10, L8, L9: 100uH, Resistors_ThroughHole:R_Axial_DIN0204_L3.6mm_D1.6mm_P7.62mm_Horizontal
- removed Q14: SC2314, TO_SOT_Packages_THT:TO-126_Horizontal
- removed R104, R106, R107: 100, TTG:R_1206_0603
- removed R105: 5.1k, TTG:R_1206_0603
- removed T16: FEEDBACK, TTG:TF_2
- removed T17: Transformer, TTG:TF14
- R103: value 5.1k -> 100
- moved C62 45.2 mm to (90.5, 70.4), turned to 90 degrees
- moved R95 39.0 mm to (114.6, 76.5), turned to 90 degrees
- moved C61 34.3 mm to (137.4, 66.6), turned to 90 degrees
- moved R79 34.1 mm to (117.3, 76.5)
- moved C27 30.0 mm to (107.1, 119.1)
- moved C56 29.6 mm to (111.9, 76.5)
- moved R78 27.3 mm to (123.0, 80.0), turned to 0 degrees
- moved U9 26.5 mm to (120.2, 70.8)
- moved T15 26.4 mm to (125.8, 72.0)
- moved U8 26.4 mm to (137.4, 70.8)
- moved R97 25.9 mm to (121.7, 75.0)
- moved T14 24.1 mm to (129.8, 85.0)
- moved C60 23.7 mm to (115.0, 70.8), turned to 180 degrees
- moved T9 23.3 mm to (134.7, 92.5), turned to 270 degrees
- moved C1 20.8 mm to (150.5, 106.0), turned to 0 degrees
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Connections:
- C33 pad 2: Net-(C30-Pad2) -> Net-(C33-Pad2)
- C56 pad 2: Net-(C30-Pad2) -> Net-(C56-Pad2)
- C62 pad 1: Net-(C62-Pad1) -> +12V
- C62 pad 2: Net-(C62-Pad2) -> GND
- R103 pad 1: Net-(C40-Pad2) -> Net-(R103-Pad1)
- R103 pad 2: Net-(L8-Pad2) -> Net-(C33-Pad2)
- R75 pad 2: Net-(C30-Pad2) -> Net-(C33-Pad2)
- R76 pad 1: Net-(C30-Pad2) -> Net-(C33-Pad2)
- R78 pad 1: Net-(R78-Pad1) -> Net-(C56-Pad2)
- R79 pad 2: Net-(R78-Pad1) -> Net-(C56-Pad2)
- R95 pad 1: Net-(R78-Pad1) -> Net-(C56-Pad2)
- U7 pad 4: Net-(C30-Pad2) -> Net-(R103-Pad1)
Routing:
- net GND: track 35.7 -> 1526.7 mm, vias 17 -> 395
- net RF: track 8.74 -> 187.7 mm, vias 0 -> 3
- net +6V: track 130.3 -> 225.4 mm, vias 4 -> 3
- net +12V: track 90.2 -> 156.8 mm
- net LO: track 9.78 -> 71.2 mm, vias 0 -> 2
- net IF: track 124.7 -> 173.9 mm, vias 1 -> 2
- net VXO: track 36.7 -> 66.9 mm, vias 2 -> 4
- net Net-(C48-Pad2): track 13.7 -> 43.4 mm
- net Net-(C63-Pad2): track 25.6 -> 0.00 mm
- net Net-(T4-Pad4): track 3.07 -> 27.8 mm
- net RX: track 63.7 -> 40.2 mm
- net Net-(D9-Pad1): track 22.4 -> 0.00 mm
- net Net-(C65-Pad1): track 22.0 -> 0.00 mm
- net Net-(C30-Pad2): track 18.4 -> 0.00 mm
- net Net-(C56-Pad2): track 0.00 -> 16.0 mm
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Other:
- board text added: "12dB"
- board text added: "2 TONE"
- board text added: "24dB"
- board text added: "2dB"
- board text added: "32dB"
- board text added: "3dB"
- board text added: "6dB"
- board text added: "IF"
- board text added: "IF AMP"
- board text added: "RF"
- board text added: "RF IN AMP"
- board text added: "VFO"

Commit message: att fixed values
Parts:
- C19, C31: value 100nF -> 10nF
Changed lines of the file:
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@@
       (effects (font (size 1 1) (thickness 0.15)))
     )
-    (fp_text value 100nF (at 0 1.9 180) (layer F.Fab) hide
+    (fp_text value 10nF (at 0 1.9 180) (layer F.Fab) hide
       (effects (font (size 1 1) (thickness 0.15)))
     )
@@
       (effects (font (size 1 1) (thickness 0.15)))
     )
-    (fp_text value 100nF (at 0 1.9 270) (layer F.Fab) hide
+    (fp_text value 10nF (at 0 1.9 270) (layer F.Fab) hide
       (effects (font (size 1 1) (thickness 0.15)))
     )
@@
   (segment (start 77.025 37) (end 76.8 37.225) (width 0.25) (layer F.Cu) (net 1))
   (via (at 76.8 37.225) (size 0.6) (drill 0.4) (layers F.Cu B.Cu) (net 1))
-  (segment (start 77.025 37) (end 78.3 37) (width 0.25) (layer F.Cu) (net 1) (status 800000))
+  (segment (start 77.025 37) (end 78.3 37) (width 0.25) (layer F.Cu) (net 1))
   (via (at 72.825 37.225) (size 0.6) (drill 0.4) (layers F.Cu B.Cu) (net 1))
   (segment (start 82.5 40.975) (end 79.425 40.975) (width 0.25) (layer B.Cu) (net 1))
@@
   (segment (start 78.325 57.35) (end 82.175 57.35) (width 0.25) (layer F.Cu) (net 1))
   (via (at 82.175 57.35) (size 0.6) (drill 0.4) (layers F.Cu B.Cu) (net 1))
-  (segment (start 85.95 57.35) (end 85.95 59) (width 0.25) (layer F.Cu) (net 1) (status 800000))
+  (segment (start 85.95 57.35) (end 85.95 59) (width 0.25) (layer F.Cu) (net 1))
   (via (at 85.95 57.35) (size 0.6) (drill 0.4) (layers F.Cu B.Cu) (net 1))
   (segment (start 82.175 57.35) (end 85.95 57.35) (width 0.25) (layer B.Cu) (net 1))
@@
   (via (at 82.5 40.975) (size 0.6) (drill 0.4) (layers F.Cu B.Cu) (net 1))
   (segment (start 82.55 41.025) (end 82.5 40.975) (width 0.25) (layer B.Cu) (net 1))
-  (segment (start 85.95 44.704) (end 85.95 41.025) (width 0.25) (layer F.Cu) (net 1) (status 400000))
+  (segment (start 85.95 44.704) (end 85.95 41.025) (width 0.25) (layer F.Cu) (net 1))
   (segment (start 85.95 41.025) (end 85.975 41.025) (width 0.25) (layer B.Cu) (net 1))
   (via (at 85.95 41.025) (size 0.6) (drill 0.4) (layers F.Cu B.Cu) (net 1))
@@
   (segment (start 85.95 52.025) (end 82.525 52.025) (width 0.25) (layer B.Cu) (net 1))
   (via (at 85.95 52.025) (size 0.6) (drill 0.4) (layers F.Cu B.Cu) (net 1))
-  (segment (start 85.95 55.704) (end 85.95 52.025) (width 0.25) (layer F.Cu) (net 1) (status 400000))
+  (segment (start 85.95 55.704) (end 85.95 52.025) (width 0.25) (layer F.Cu) (net 1))
   (segment (start 82.5 52) (end 82.5 52.025) (width 0.25) (layer F.Cu) (net 1))
   (via (at 82.5 52) (size 0.6) (drill 0.4) (layers F.Cu B.Cu) (net 1))
@@
   (segment (start 82.5 63) (end 79.325 63) (width 0.25) (layer B.Cu) (net 1))
   (via (at 82.5 63) (size 0.6) (drill 0.4) (layers F.Cu B.Cu) (net 1))
-  (segment (start 85.95 66.704) (end 85.95 63) (width 0.25) (layer F.Cu) (net 1) (status 400000))
+  (segment (start 85.95 66.704) (end 85.95 63) (width 0.25) (layer F.Cu) (net 1))
   (via (at 85.95 63) (size 0.6) (drill 0.4) (layers F.Cu B.Cu) (net 1))
   (segment (start 82.5 63) (end 85.95 63) (width 0.25) (layer B.Cu) (net 1))
@@
   (segment (start 82.125 68.325) (end 85.95 68.325) (width 0.25) (layer B.Cu) (net 1))
   (via (at 85.95 68.325) (size 0.6) (drill 0.4) (layers F.Cu B.Cu) (net 1))
-  (segment (start 85.95 68.325) (end 85.95 70) (width 0.25) (layer F.Cu) (net 1) (status 800000))
+  (segment (start 85.95 68.325) (end 85.95 70) (width 0.25) (layer F.Cu) (net 1))
   (via (at 82.125 68.325) (size 0.6) (drill 0.4) (layers F.Cu B.Cu) (net 1))
   (segment (start 78.3 68.325) (end 82.125 68.325) (width 0.25) (layer F.Cu) (net 1))
@@
   (segment (start 85.95 74) (end 82.5 74) (width 0.25) (layer B.Cu) (net 1))
   (via (at 82.5 74) (size 0.6) (drill 0.4) (layers F.Cu B.Cu) (net 1))
-  (segment (start 85.95 77.704) (end 85.95 74) (width 0.25) (layer F.Cu) (net 1) (status 400000))
+  (segment (start 85.95 77.704) (end 85.95 74) (width 0.25) (layer F.Cu) (net 1))
   (via (at 73.175 73.9) (size 0.6) (drill 0.4) (layers F.Cu B.Cu) (net 1))
   (segment (start 75.575 73.9) (end 73.175 73.9) (width 0.25) (layer B.Cu) (net 1))
@@
   (segment (start 75.475 79.35) (end 75.5 79.35) (width 0.25) (layer F.Cu) (net 1))
   (via (at 75.475 79.35) (size 0.6) (drill 0.4) (layers F.Cu B.Cu) (net 1))
-  (segment (start 85.95 81) (end 85.95 79.35) (width 0.25) (layer F.Cu) (net 1) (status 400000))
+  (segment (start 85.95 81) (end 85.95 79.35) (width 0.25) (layer F.Cu) (net 1))
   (segment (start 85.95 79.35) (end 85.925 79.35) (width 0.25) (layer B.Cu) (net 1))
   (via (at 85.95 79.35) (size 0.6) (drill 0.4) (layers F.Cu B.Cu) (net 1))
