File: TTG.sch (KiCad schematic (older format))
At the start: 231 parts, among them J1 RF_In, J10 Conn_01x01, J11 Conn_01x01, J12 Conn_01x01, J13 Conn_01x01, J14 RF_In, J15 IF, J16 RX/TX, J2 Jack-DC, J3 RF_In, J4 RF_In, J5 RF_In, J6 RF_In, J7 RF_In, J8 OFF, J9 OFF, Q1 MMBT9018, Q10 MMBTFJ310, Q11 SI2301-TP, Q12 SI2301-TP, Q2 MMBT9018, Q3 MMBT9018, Q4 MMBT9018, Q5 SS9018, Q6 MMBTFJ310, Q7 MMBTFJ310, Q8 MMBTFJ310, Q9 MMBTFJ310, SW1 SW_DPDT_x2, SW2 SW_DPDT_x2, SW3 SW_DPDT_x2, SW4 SW_DPDT_x2, SW5 SW_DPDT_x2, SW6 SW_DPDT_x2, SW7 SW_DPDT_x2, SW8 SW_DPDT_x2, T1 Transformer, T10 Transformer_1P_2S, T11 Transformer, T12 Transformer_1P_1S, T13 Transformer, T2 Transformer, T3 Transformer_1P_1S, T4 Transformer_1P_2S, T5 Transformer_1P_2S, T6 Transformer_1P_2S, T7 Transformer_1P_2S, T8 Transformer_1P_2S, T9 Transformer_1P_2S, U1 L7809, U2 NC7WZ14, U3 FSA3157L6X, U4 FSA3157L6X, U5 LM317L_TO92, U6 L78L05_TO92, U7 FSA3157L6X, U8 FSA3157L6X, Y1 Crystal_GND23, Y2 Crystal_GND23

Commit message: SC2314
Parts:
- removed C30: 10uF, Capacitors_Tantalum_SMD:CP_Tantalum_Case-A_EIA-3216-18_Hand, symbol CP_Small
- removed T10, T9: Transformer_1P_2S, TTG:HF_transf3, symbol Transformer_1P_2S
- added C30, C56, C57, C58, C59, C60, C61, C62, C63, C64, C65, C66, C67, C68: 100nF, TTG:C_1206_0603, symbol C_Small
- added D10, D9: LL4148, Diodes_SMD:D_MiniMELF_Handsoldering, symbol D_Small
- added L10, L8, L9: 100uH, Resistors_ThroughHole:R_Axial_DIN0204_L3.6mm_D1.6mm_P7.62mm_Horizontal, symbol L_Small
- added Q13: BF998, TO_SOT_Packages_SMD:SOT-143_Handsoldering, symbol BF998
- added Q14: SC2314, TO_SOT_Packages_THT:TO-126_Horizontal, symbol Q_NPN_ECB
- added R100, R102: 100R, TTG:R_1206_0603, symbol R_Small
- added R101: 2.2k, Resistors_SMD:R_1206_HandSoldering, symbol R_Small
- added R103, R105: 5.1k, TTG:R_1206_0603, symbol R_Small
- added R104, R106, R107, R96, R97: 100, TTG:R_1206_0603, symbol R_Small
- added R95: 1k, TTG:R_1206_0603, symbol R_Small
- added R98: 470, TTG:R_1206_0603, symbol R_Small
- added R99: 27k, TTG:R_1206_0603, symbol R_Small
- added T10: N7ZWY1_4, TTG:N7ZWY, symbol N7ZWY1_4
- added T14, T15: Transformer_1P_2S, TTG:HF_transf3, symbol Transformer_1P_2S
- added T16: FEEDBACK, TTG:TF_2, symbol Transformer_1P_1S
- added T17: Transformer, TTG:TF14, symbol Transformer
- added T9: Transformer_1P_1S, TTG:TF14, symbol Transformer_1P_1S
- added U9: FSA3157L6X, TO_SOT_Packages_SMD:SOT-363_SC-70-6_Handsoldering, symbol FSA3157L6X
- C14: footprint RX998:C_1206_0603 -> Capacitors_SMD:C_1206_HandSoldering
- D1: footprint (none) -> Diodes_ThroughHole:D_DO-41_SOD81_P7.62mm_Horizontal
- D6, D7: footprint (none) -> Diodes_SMD:D_MiniMELF_Handsoldering
- D8: value D_Small -> LL4148; footprint (none) -> Diodes_SMD:D_MiniMELF_Handsoldering
- J16: footprint (none) -> Pin_Headers:Pin_Header_Straight_1x02_Pitch2.54mm
- Q11, Q12: footprint (none) -> TO_SOT_Packages_SMD:SOT-23_Handsoldering
- R75, R76: value 100 -> 1k
- R78: value 10k -> 100
- R79: value 10k -> 1k
- T12: value Transformer_1P_1S -> FEEDBACK; footprint (none) -> TTG:TF_2
Connections:
- net +12V: now also R100.1
- net +6V: now also R75.1, R79.1, C60.1, C61.1, U9.5 (V+); no longer R78.1
- net GND: now also C33.1, R76.2, T12.1 (AA), C30.1, C56.1, C57.1, C58.1, C59.2, C60.2, C61.2, C65.2, C66.2, C67.2, C68.2, L8.1, R102.2, R105.2, R95.2, R98.2, R99.2, T14.2 (AB), T15.2 (AB), T16.1 (AA), U9.2 (GND); no longer C33.2, R79.2, T12.2 (AB)
- net IF: now also Q13.2 (D), R101.2, T14.1 (AA), T9.2 (AB), T9.4 (SB)
- net LO: now also R96.2, R97.2; no longer R76.2
- net RF: now also Q13.4 (G1), R99.1, T10.2, T10.7, T15.1 (AA)
- net RX: now also C68.1, L10.2
- net TX: now also C67.1, L9.2
- net VXO: now also Q13.3 (G2), R98.1
- net at U7.1: now also T10.5, T9.3 (SA); no longer U8.3
- net at C34.2: now also T10.1, T10.8
- net at U7.3: now also T10.3, T9.1 (AA); no longer U8.1
- net at U8.4: now also T14.3 (SA)
- net at R76.1: now also C33.2, R75.2, U7.4, C30.2, C56.2; no longer U8.6
- net at C43.1, C44.1, C45.1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: now also T12.3 (SA); no longer T12.4 (SB)
- net at C48.2, J15.1 (In): now also T12.2 (AB), C64.2, T16.2 (AB); no longer T12.1 (AA)
- net at C42.2, L5.2, R81.1: now also T12.4 (SB); no longer T12.3 (SA)
- net at C40.2, J14.1 (In): now also R103.1, T16.4 (SB)
- new net: T10.4, T10.6
- new net: T15.6 (SD), U8.1, U9.3
- new net: T15.3 (SA), U8.3, U9.1
- new net: R96.1, U8.6
- new net: C57.2, T15.4 (SB), T15.5 (SC)
- new net: R78.2, T14.4 (SB), T14.5 (SC)
- new net: T14.6 (SD), U9.4
- new net: R78.1, R79.2, R95.1
- new net: R97.1, U9.6
- new net: C59.1, Q13.1 (S), R102.1
- new net: C58.2, R100.2, R101.1
- new net: Q14.1 (E), R104.1
- new net: D9.1 (K), Q14.2 (C), R106.1, T17.1 (AA)
- new net: C63.1, Q14.3 (B), R105.1, R107.2
- new net: C64.1, T17.2 (AB), T17.3 (SB)
- new net: C63.2, D10.1 (K), R107.1, T17.4 (SA)
- new net: C62.2, R106.2
- new net: C62.1, R104.2, T16.3 (SA)
- new net: L8.2, R103.2
- new net: C66.1, D9.2 (A), L9.1
- new net: C65.1, D10.2 (A), L10.1
Other:
- moved on the sheet: C14, C15, C17, C20, C21, C22, C23, C24, C25, C26, C27, C29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

Commit message: release, no rasin mixer
Parts:
- removed C30, C63, C64, C65, C66, C67, C68: 100nF, TTG:C_1206_0603, symbol C_Small
- removed D10, D9: LL4148, Diodes_SMD:D_MiniMELF_Handsoldering, symbol D_Small
- removed L10, L8, L9: 100uH, Resistors_ThroughHole:R_Axial_DIN0204_L3.6mm_D1.6mm_P7.62mm_Horizontal, symbol L_Small
- removed Q14: SC2314, TO_SOT_Packages_THT:TO-126_Horizontal, symbol Q_NPN_ECB
- removed R104, R106, R107: 100, TTG:R_1206_0603, symbol R_Small
- removed R105: 5.1k, TTG:R_1206_0603, symbol R_Small
- removed T16: FEEDBACK, TTG:TF_2, symbol Transformer_1P_1S
- removed T17: Transformer, TTG:TF14, symbol Transformer
- R103: value 5.1k -> 100
Connections:
- net +12V: now also C62.1
- net GND: now also C62.2
- net at C33.2, R75.2, R76.1: now also R103.2; no longer C56.2, U7.4
- net at C40.2, J14.1 (In): no longer R103.1
- net at R78.1, R79.2, R95.1: now also C56.2
- new net: R103.1, U7.4
Other:
- moved on the sheet: C33, C56, R75, R76

Commit message: att fixed values
Parts:
- C11, C8: value 100 -> 200
- C18, C19, C31: value 100nF -> 10nF
- R10, R15, R42, R5: value 33 -> 18k
- R14, R8: value 68 -> 82
- R16, R24: value 33 -> 680
- R17, R25: value 33 -> 1k2
- R20: value 68 -> 12
- R21: value 68 -> 360
- R27, R31: value 33 -> 11k
- R28, R32: value 33 -> 300
- R29: value 68 -> 18
- R30: value 68 -> 820
- R33, R38: value 33 -> 180
- R34, R35, R39, R4, R41, R9: value 33 -> 910
- R36: value 68 -> 47
- R37: value 68 -> 180
- R40, R7: value 68 -> 6.2
- R43, R47: value 33 -> 1k
- R44, R48, R49, R53: value 33 -> 91
- R45: value 68 -> 100
- R46: value 68 -> 1k2
- R52: value 68 -> 4k7

Commit message: attenuators values update
Parts:
- R50, R54: value 33 -> 150
- R51: value 68 -> 430
- R55, R59, R61, R65: value 33 -> 56
- R56, R60, R62, R66: value 33 -> 820
- R57, R63: value 68 -> 180k
- R58, R64: value 68 -> 1k
Other:
- moved on the sheet: C14, C15, C17, C20, C21, C22, C23, C24, C25, C26, C27, C29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
